File: PCBs/SAME54-Dev.sch (EAGLE design)
At the start: 109 parts, among them J2 USB_A_FEMALE, Q2 TRANS_NPN-MMBTA42, SW1 MOMENTARY-SWITCH-SPST-SMD-6.2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, SW2 MOMENTARY-SWITCH-SPST-SMD-6.2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, SW3 MOMENTARY-SWITCH-SPST-SMD-6.2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, U1 ATSAME54N20A, U2 KSZ8091RNA, U3 AP1117, U4 CP2102, U5 W25N01GV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

Commit message: Added schematic PDF
Parts:
- removed U$1: SI-50170-F, conn-custom:SI-50170-F
- removed U$2: DM3D-SF, conn-custom:DM3D-SF
- added X2: SI-50170-F, conn-custom:SI-50170-F
- added X4: DM3D-SF, conn-custom:DM3D-SF
Connections:
- net +3V3: now also X2.LEDG+, X2.LEDY+, X4.VDD; no longer U$1.LEDG+, U$1.LEDY+, U$2.VDD
- net ETH-LED-G-: now also X2.LEDG-; no longer U$1.LEDG-
- net ETH-LED-Y-: now also X2.LEDY-; no longer U$1.LEDY-
- net GND: now also X4.CD2, X4.SHIELD, X4.VSS; no longer U$2.CD2, U$2.SHIELD, U$2.VSS
- net MCI_CD: now also X4.CD1; no longer U$2.CD1
- net MCI_CMD: now also X4.CMD; no longer U$2.CMD
- net MCI_D0: now also X4.DAT0; no longer U$2.DAT0
- net MCI_D1: now also X4.DAT1; no longer U$2.DAT1
- net MCI_D2: now also X4.DAT2; no longer U$2.DAT2
- net MCI_D3: now also X4.CD/DAT3; no longer U$2.CD/DAT3
- net MCI_SDCK: now also X4.CLK; no longer U$2.CLK
- net N$6: now also X2.TCT; no longer U$1.TCT
- net N$7: now also X2.RCT; no longer U$1.RCT
- net RJ45-GND: now also X2.GND, X2.SHIELD; no longer U$1.GND, U$1.SHIELD
- net RX_N: now also X2.RD-; no longer U$1.RD-
- net RX_P: now also X2.RD+; no longer U$1.RD+
- net TX_N: now also X2.TD-; no longer U$1.TD-
- net TX_P: now also X2.TD+; no longer U$1.TD+
Other:
- note added: "100 ohm differential"
- note added: "Ethernet PHY"
- note added: "I/O Header"
- note added: "ISP Header"
- note added: "Indicator LEDs"
- note added: "MCU IO Banks"
- note added: "MCU Power and Reset"
- note added: "Micro SD SDHC Interface"
- note added: "Oscillator"
- note added: "Push Buttons"
- note added: "QSPI Interface and Flash Chip"
- note added: "USB Power, ESD and OTG Host Detection"
- note added: "USB to Serial CP2102"
- note added: "Voltage Regulator 3.3V"
- note removed: "100 ohm differential JLC7628"
